File: stripline-pickup-a.kicad_pcb (KiCad board)
At the start: 4 copper layers, 300 x 240 mm, 11 parts

Commit message: stripline width modified and routed to samtec connectors.
Parts:
- moved SC2 25.4 mm to (437.0, 272.0)
- moved SC1 25.4 mm to (79.6, 181.0)
- moved SL1 7.26 mm to (143.8, 123.8)
Routing:
- net Net-(SC2-Pad136): track 0.00 -> 96.9 mm
- net Net-(SC2-Pad20): track 0.00 -> 95.1 mm
- net Net-(SC2-Pad132): track 0.00 -> 92.2 mm
- net Net-(SC2-Pad24): track 0.00 -> 90.2 mm
- net Net-(SC2-Pad28): track 0.00 -> 87.7 mm
- net Net-(SC2-Pad128): track 0.00 -> 87.2 mm
- net Net-(SC2-Pad124): track 0.00 -> 82.4 mm
- net Net-(SC2-Pad32): track 0.00 -> 78.6 mm
- net Net-(SC2-Pad120): track 0.00 -> 77.5 mm
- net Net-(SC2-Pad44): track 0.00 -> 74.4 mm
- net Net-(SC2-Pad36): track 0.00 -> 74.2 mm
- net Net-(SC2-Pad116): track 0.00 -> 73.4 mm
- net Net-(SC2-Pad56): track 0.00 -> 72.5 mm
- net Net-(SC2-Pad40): track 0.00 -> 71.0 mm
- net Net-(SC2-Pad104): track 0.00 -> 70.1 mm
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Other:
- board size 300 x 240 mm -> 351.2 x 240 mm
